File: hardware/flute.kicad_pcb (KiCad board)
At the start: 2 copper layers, 230 x 20 mm, 47 parts, among them J1 Conn_01x02, J3 Conn_01x04, SW1 C, SW2 D, SW3 E, SW4 F, SW5 G, SW6 A, SW7 H, SW8 OCTAVE?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

Commit message: pcb ver1.1
Parts:
- moved C5 0.52 mm to (58.2, 103.7)
- moved TP6 0.25 mm to (68.3, 113.9)
- moved C4 0.23 mm to (50.4, 118.0)
- moved C16 0.22 mm to (48.7, 118.0)
- moved TP8 0.13 mm to (36.1, 104.5)
- moved C7 0.11 mm to (52.1, 118.0)
- moved C14 0.07 mm to (45.2, 110.0)
Other:
- board text added: "KN HARDWIRE ELECTRONIC FLUTE VER 1.1 AGH UNIVERSITY OF CRACOW 2025"
- board text removed: "KN HARDWIRE ELECTRONIC FLUTE VER 1.0 AGH UNIVERSITY OF CRACOW 2025"

Commit message: complete pcb ver1.1
Parts:
- moved JP2 3.58 mm to (258.7, 103.7)
- moved R2 3.46 mm to (255.3, 107.0), turned to 180 degrees
- moved JP1 3.14 mm to (255.4, 103.7), turned to 90 degrees
- moved C2 3.05 mm to (258.6, 106.3), turned to 0 degrees
Routing:
- net Net-(J1-Pin_1): track 9.25 -> 6.14 mm
- net /PWM_OUT: track 208.7 -> 206.6 mm
- net Net-(JP1-A): track 8.17 -> 6.49 mm
